File: ram.kicad_sch (KiCad schematic)
At the start: 87 parts, among them J1 DIN41612_01x32_A, J2 DIN41612_01x32_B, J3 DIN41612_01x32_C

Commit message: WIP: 8MB 72 pin SIMM to Altos 8MB RAM module
Parts:
- removed C1, C13, C17, C22, C23, C24, C25, C3, C6, C7, C9: C, symbol Device:C_Polarized
- removed C11, C12, C16, C20, C5: C, symbol Device:C
- removed C2, C21, C26, C8: 4.5n, symbol Device:C
- removed R10, R11, R13, R14, R15, R17, R18, R19, R20, R4, R7, R8, R9: 27, symbol Device:R
- removed RN1, RN10, RN3, RN4, RN6, RN8: 22, Resistor_THT:R_Array_SIP10, symbol Device:R_Pack05_SIP
- removed SIM1, SIM2, SIM3, SIM4, SIM5, SIM6, SIM7, SIM8: ~, symbol chips:SIMM_1X30_PIN
- removed U1, U5, U6, U7, U8: ~, symbol chips:SN54AS1004A
- removed U10, U9: ~, symbol chips:SN74AS1000A
- added U13: ~, symbol chips:SIMM_1X72_PIN
Connections:
- net O_S12A6 is gone; now on net ~{RAS_OE}: U2.4 (2Y)
- net O_S12A7 is gone; now on net ~{CAS_OE}: U2.6 (3Y)
- net S34A0 is gone; now on net ~{A0}: RN7.4 (R2.2)
- net S34A1 is gone; now on net ~{A1}: RN7.6 (R3.2)
- net S34A2 is gone; now on net ~{A2}: RN7.8 (R4.2)
- net S34A3 is gone; now on net ~{A3}: RN7.10 (R5.2)
- net S34A4 is gone; now on net ~{A4}: RN9.2 (R1.2)
- net S34A5 is gone; now on net ~{A5}: RN9.4 (R2.2)
- net S34A6 is gone; now on net ~{A6}: RN9.6 (R3.2)
- net S34A7 is gone; now on net ~{A7}: RN9.8 (R4.2)
- net S34A8 is gone; now on net ~{A8}: RN9.10 (R5.2)
- net S34A9 is gone; now on net ~{A9}: RN7.2 (R1.2)
- net ~{O_CAS5} is gone; now on net ~{CAS2}: U11.11 (4Y)
- net ~{O_CAS7} is gone; now on net ~{WE}: R3.1
- net ~{O_RAS1} is gone; now on net ~{O_RAS2}: R1.1
- net ~{O_RAS3} is gone; now on net ~{CAS1}: U11.6 (2Y)
- net ~{O_RAS5} is gone; now on net ~{CAS3}: U11.8 (3Y)
- net ~{RAS1} is gone; now on net ~{RAS2}: R1.2
- net A05: no longer U2.1 (1A)
- net A06: no longer U2.3 (2A)
- net A07: no longer U2.5 (3A)
- net A08: no longer U2.9 (4A)
- net CAS0: now also U11.2 (1B); no longer U12.2 (1B)
- net CAS1: now also U11.5 (2B); no longer U11.2 (1B)
- net CAS2: now also U11.13 (4B); no longer U12.13 (4B)
- net CAS3: now also U11.10 (3B); no longer U11.13 (4B)
- net CAS_OE: now also U11.4 (2A), U11.9 (3A), U2.5 (3A); no longer U12.1 (1A), U12.12 (4A), U4.12 (6Y)
- net D00: now also U13.2 (D00)
- net D01: now also U13.4 (D01)
- net D02: now also U13.6 (D02)
- net D03: now also U13.8 (D03)
- net D04: now also U13.20 (D04)
- net D05: now also U13.22 (D05)
- net D06: now also U13.24 (D06)
- net D07: now also U13.26 (D07)
- net D08: now also U13.49 (D08)
- net D09: now also U13.51 (D09)
- net D10: now also U13.53 (D10)
- net D11: now also U13.55 (D11)
- net D12: now also U13.57 (D12)
- net D13: now also U13.61 (D13)
- net D14: now also U13.63 (D14)
- net D15: now also U13.65 (D15)
- net D16: now also U13.3 (D16)
- net D17: now also U13.5 (D17)
- net D18: now also U13.7 (D18)
- net D19: now also U13.9 (D19)
- net D20: now also U13.21 (D20)
- net D21: now also U13.23 (D21)
- net D22: now also U13.25 (D22)
- net D23: now also U13.27 (D23)
- net D24: now also U13.50 (D24)
- net D25: now also U13.52 (D25)
- net D26: now also U13.54 (D26)
- net D27: now also U13.56 (D27)
- net D28: now also U13.58 (D28)
- net D29: now also U13.60 (D29)
- net D30: now also U13.62 (D30)
- net D31: now also U13.64 (D31)
- net GND: now also U13.1 (GND), U13.39 (GND), U13.72 (GND)
- net P0: now also U13.36 (P00)
- net P1: now also U13.37 (P01)
- net P2: now also U13.35 (P02)
- net P3: now also U13.38 (P03)
- net RAS0: now also U12.2 (1B)
- net RAS1: no longer U11.10 (3B), U11.5 (2B), U12.10 (3B)
- net RAS_OE: now also U12.1 (1A), U2.3 (2A); no longer U11.4 (2A), U11.9 (3A), U12.9 (3A), U4.10 (5Y)
- net VCC: now also U13.10 (VCC), U13.30 (VCC), U13.59 (VCC)
- net WE: now also U2.1 (1A)
- net ~{CAS0}: now also U11.3 (1Y)
- net ~{CAS_OE}: no longer U4.13 (6A)
- net ~{O_CAS0}: now also U13.40 (~{CAS0})
- net ~{O_CAS1}: now also U13.43 (~{CAS1})
- net ~{O_CAS2}: now also U13.41 (~{CAS2}); no longer U12.3 (1Y)
- net ~{O_CAS3}: now also U13.42 (~{CAS3}); no longer U11.3 (1Y)
- net ~{O_RAS0}: now also U13.34 (~{RAS2}), U13.44 (~{RAS0})
- net ~{O_RAS2}: now also U13.33 (~{RAS3}), U13.45 (~{RAS1}); no longer U12.6 (2Y)
- net ~{RAS0}: now also U12.3 (1Y)
- net ~{RAS2}: now also U12.6 (2Y)
- net ~{RAS_OE}: no longer U4.11 (5A)
- net O_S12A5 renamed ~{WE}
- net O_S12A8: no longer names the net of U2.8 (4Y)
- net O_S34A0 renamed ~{A0}
- net ~{A0}: no longer RN7.3 (R2.1)
- net O_S34A1 renamed ~{A1}
- net ~{A1}: no longer RN7.5 (R3.1)
- net O_S34A2 renamed ~{A2}
- net ~{A2}: no longer RN7.7 (R4.1)
- net O_S34A3 renamed ~{A3}
- net ~{A3}: no longer RN7.9 (R5.1)
- net O_S34A4 renamed ~{A4}
- net ~{A4}: no longer RN9.1 (R1.1)
- net O_S34A5 renamed ~{A5}
- net ~{A5}: no longer RN9.3 (R2.1)
- net O_S34A6 renamed ~{A6}
- net ~{A6}: no longer RN9.5 (R3.1)
- net O_S34A7 renamed ~{A7}
- net ~{A7}: no longer RN9.7 (R4.1)
- net O_S34A8 renamed ~{A8}
- net ~{A8}: no longer RN9.9 (R5.1)
- net O_S34A9 renamed ~{A9}
- net ~{A9}: no longer RN7.1 (R1.1)
- net ~{CAS7} renamed ~{O_WE}
- net ~{O_WE}: now also U13.47 (~{WE})
- net ~{O_CAS4}: no longer names the net of U12.11 (4Y)
- net ~{O_RAS4}: no longer names the net of U12.8 (3Y)
- new net ~{O_A0}: RN7.3 (R2.1), U13.12 (A00)
- new net ~{O_A1}: RN7.5 (R3.1), U13.13 (A01)
- new net ~{O_A2}: RN7.7 (R4.1), U13.14 (A02)
- new net ~{O_A3}: RN7.9 (R5.1), U13.15 (A03)
- new net ~{O_A4}: RN9.1 (R1.1), U13.16 (A04)
- new net ~{O_A5}: RN9.3 (R2.1), U13.17 (A05)
- new net ~{O_A6}: RN9.5 (R3.1), U13.18 (A06)
- new net ~{O_A7}: RN9.7 (R4.1), U13.28 (A07)
- new net ~{O_A8}: RN9.9 (R5.1), U13.31 (A08)
- new net ~{O_A9}: RN7.1 (R1.1), U13.32 (A09)
- no-connect marks 30 -> 26
Other:
- note removed: "BANK 0"
- note removed: "BANK 1"
- note removed: "BYTE 0"
- note removed: "BYTE 1"
- note removed: "BYTE 2"
- note removed: "BYTE 3"
- moved on the sheet: R12, R16, R2, R21, R22, R23, R24, R5, R6, RN11, RN12, RN13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
